Commit message: fixed mass and a bit better inertia
Former-commit-id: af073f24fed056738a268f3bf9a55483404e630c

File: xacro/bobble_chassis.urdf.xacro (robot description, xacro)
@@ -5,6 +5,6 @@
   		<inertial>
 	  		<origin xyz="-0.06 0.0 0.180" rpy="0.0 0.0 0.0"/>
-  	  		<mass value="10.0"/>
-	  		<inertia ixx="0.0416666666" ixy="0.0" ixz="0.0" iyy="0.1416666666" iyz="0.0" izz="0.1666666666"/>
+  	  		<mass value="2.043"/>
+	  		<inertia ixx="0.03" ixy="0.0" ixz="0.0" iyy="0.03" iyz="0.0" izz="0.03"/>
 		</inertial>
 		<visual>

File: xacro/left_wheel.urdf.xacro (robot description, xacro)
@@ -4,6 +4,6 @@
 	<link name="left_wheel_link">
 		<inertial>
-			<mass value="10.0"/>
-			<inertia ixx="0.02708333333" ixy="0.0" ixz="0.0" iyy="0.02708333333" iyz="0.0" izz="0.05"/>
+			<mass value="0.084"/>
+			<inertia ixx="0.00035" ixy="0.0" ixz="0.0" iyy="0.00035" iyz="0.0" izz="0.00035"/>
 		</inertial>
 		<visual>
@@ -24,13 +24,12 @@
 		<selfCollide>true</selfCollide>
 	</gazebo>
-	<joint name="left_wheel_hinge" type="revolute">
+	<joint name="left_wheel_hinge" type="continuous">
 		<parent link="${parent}"/>
 		<child link="left_wheel_link"/>
 		<origin rpy="0 0 0" xyz="0.0 0.1 0.05"/>
 		<axis xyz="0 1 0"/>
-		<limit effort="30" lower="-1000.0" upper="1000.0" velocity="2.0"/>
 		<!-- <safety_controller k_velocity="0.5"/> -->
 		<!-- <joint_properties damping="100.0" friction="1000.0" /> -->
-    	<dynamics damping="0.9" friction="${3.0/7}"/>
+    	<dynamics damping="0.0" friction="0.0"/>
 	</joint>
 	<transmission name="left_wheel_transmission">

File: xacro/right_wheel.urdf.xacro (robot description, xacro)
@@ -4,6 +4,6 @@
 	<link name="right_wheel_link">
 		<inertial>
-			<mass value="10.0"/>
-			<inertia ixx="0.02708333333" ixy="0.0" ixz="0.0" iyy="0.02708333333" iyz="0.0" izz="0.05"/>
+			<mass value="0.084"/>
+			<inertia ixx="0.00035" ixy="0.0" ixz="0.0" iyy="0.00035" iyz="0.0" izz="0.00035"/>
 		</inertial>
 		<visual>
@@ -24,13 +24,12 @@
 		<selfCollide>true</selfCollide>
 	</gazebo>
-	<joint name="right_wheel_hinge" type="revolute">
+	<joint name="right_wheel_hinge" type="continuous">
 		<parent link="${parent}"/>
 		<child link="right_wheel_link"/>
 		<origin rpy="0 0 0" xyz="0.0 -0.1 0.05"/>
 		<axis xyz="0 1 0"/>
-		<limit effort="30" lower="-1000.0" upper="1000.0" velocity="2.0"/>
 		<!-- <safety_controller k_velocity="0.5"/> -->
 		<!-- <joint_properties damping="100.0" friction="1000.0" /> -->
-		<dynamics damping="0.9" friction="${3.0/7}"/>
+		<dynamics damping="0.0" friction="0.0"/>
 	</joint>
 	<transmission name="right_wheel_transmission">

Commit message: changed center of mass to be over the center of the wheels
Former-commit-id: 2e2e1a17a98857ed74915676f24eaeec65325ad1

File: xacro/bobble_chassis.urdf.xacro (robot description, xacro)
@@ -4,5 +4,5 @@
 	<link name="bobble_chassis_link">
   		<inertial>
-	  		<origin xyz="-0.06 0.0 0.180" rpy="0.0 0.0 0.0"/>
+	  		<origin xyz="0.0 0.0 0.180" rpy="0.0 0.0 0.0"/>
   	  		<mass value="2.043"/>
 	  		<inertia ixx="0.03" ixy="0.0" ixz="0.0" iyy="0.03" iyz="0.0" izz="0.03"/>

Commit message: update offsets for new meshes and model

File: xacro/bobble_chassis.urdf.xacro (robot description, xacro)
@@ -9,13 +9,13 @@
 		</inertial>
 		<visual>
-	  		<origin xyz="0.0 0.0 0.130" rpy="0.0 0.0 0.0"/>
+	  		<origin xyz="-0.05862 0.09227 -0.022" rpy="1.5707 0.0 0.0"/>
             <geometry>
-  				<mesh filename="package://bobble_description/meshes/chassis.dae" scale="1.0 1.0 1.0"/>
+  				<mesh filename="package://bobble_description/meshes/chassis.dae" scale="0.001 0.001 0.001"/>
             </geometry>
    		</visual>
 		<collision>
-	  		<origin xyz="0.0 0.0 0.130" rpy="0.0 0.0 0.0"/>
+	  		<origin xyz="0.0 0.0 0.10263" rpy="0.0 0.0 0.0"/>
             <geometry>
-              <box size="0.1 0.11 0.185" />
+              <box size="0.122 0.1129 0.19226" />
             </geometry>
 			<contact_coefficients kd="1.0" kp="1000.0" mu="0"/>

File: xacro/left_wheel.urdf.xacro (robot description, xacro)
@@ -8,7 +8,7 @@
 		</inertial>
 		<visual>
-			<origin xyz="0.0 0.0 0.0" rpy="0.0 1.5707 1.5707"/>
+			<origin xyz="-0.0275 -0.0135 -0.0275" rpy="0.0 0.0 0.0"/>
 			<geometry name="left_wheel_link_visual">
-  				<mesh filename="package://bobble_description/meshes/wheel.dae" scale="1.0 1.0 1.0"/>
+  				<mesh filename="package://bobble_description/meshes/wheel.dae" scale="0.001 0.001 0.001"/>
 			</geometry>
   		</visual>
@@ -16,5 +16,5 @@
 			<origin xyz="0.0 0.0 0.0" rpy="0.0 1.5707 1.5707"/>
             <geometry>
-              <cylinder radius="0.05" length="0.05" />
+              <cylinder radius="0.0275" length="0.027" />
             </geometry>
 			<contact_coefficients kd="1.0" kp="1000.0" mu="0"/>
@@ -27,5 +27,5 @@
 		<parent link="${parent}"/>
 		<child link="left_wheel_link"/>
-		<origin rpy="0 0 0" xyz="0.0 0.1 0.05"/>
+		<origin rpy="0 0 0" xyz="0.0 0.06995 0.01375"/>
 		<axis xyz="0 1 0"/>
 		<!-- <safety_controller k_velocity="0.5"/> -->

File: xacro/right_wheel.urdf.xacro (robot description, xacro)
@@ -8,7 +8,7 @@
 		</inertial>
 		<visual>
-			<origin xyz="0.0 0.0 0.0" rpy="0.0 1.5707 -1.5707"/>
+			<origin xyz="0.0275 0.0135 -0.0275" rpy="0.0 0.0 3.1415926"/>
 			<geometry name="right_wheel_link_visual">
-  				<mesh filename="package://bobble_description/meshes/wheel.dae" scale="1.0 1.0 1.0"/>
+  				<mesh filename="package://bobble_description/meshes/wheel.dae" scale="0.001 0.001 0.001"/>
 			</geometry>
   		</visual>
@@ -16,5 +16,5 @@
 			<origin xyz="0.0 0.0 0.0" rpy="0.0 1.5707 -1.5707"/>
             <geometry>
-              <cylinder radius="0.05" length="0.05" />
+              <cylinder radius="0.0275" length="0.027" />
             </geometry>
 			<contact_coefficients kd="1.0" kp="1000.0" mu="0"/>
@@ -27,5 +27,5 @@
 		<parent link="${parent}"/>
 		<child link="right_wheel_link"/>
-		<origin rpy="0 0 0" xyz="0.0 -0.1 0.05"/>
+		<origin rpy="0 0 0" xyz="0.0 -0.06995 0.01375"/>
 		<axis xyz="0 1 0"/>
 		<!-- <safety_controller k_velocity="0.5"/> -->

Commit message: fixed collisions, center of masses

File: xacro/bobble_chassis.urdf.xacro (robot description, xacro)
@@ -4,5 +4,5 @@
 	<link name="bobble_chassis_link">
   		<inertial>
-	  		<origin xyz="0.0 0.0 0.180" rpy="0.0 0.0 0.0"/>
+	  		<origin xyz="0.0 0.0 0.075" rpy="0.0 0.0 0.0"/>
   	  		<mass value="2.043"/>
 	  		<inertia ixx="0.03" ixy="0.0" ixz="0.0" iyy="0.03" iyz="0.0" izz="0.03"/>
@@ -17,7 +17,7 @@
 	  		<origin xyz="0.0 0.0 0.10263" rpy="0.0 0.0 0.0"/>
             <geometry>
-              <box size="0.122 0.1129 0.19226" />
+              <box size="0.075 0.1129 0.19226" />
             </geometry>
-			<contact_coefficients kd="1.0" kp="1000.0" mu="0"/>
+			<contact_coefficients kd="10.0" kp="1000.0" mu="10.0"/>
 		</collision>
 	</link>

File: xacro/camera.urdf.xacro (robot description, xacro)
@@ -11,5 +11,5 @@
 	  <link name="camera_link">
 		  <collision>
-			  <origin xyz="0 0 0" rpy="0 0 0"/>
+			  <origin xyz="0 0 0.18" rpy="0 0 0"/>
 			  <geometry>
 				  <box size="${camera_link} ${camera_link} ${camera_link}"/>
@@ -25,5 +25,5 @@
 		  <inertial>
 			  <mass value="1e-5" />
-			  <origin xyz="0 0 0" rpy="0 0 0"/>
+			  <origin xyz="0 0 0.18" rpy="0 0 0"/>
 			  <inertia ixx="1e-6" ixy="0" ixz="0" iyy="1e-6" iyz="0" izz="1e-6" />
 		  </inertial>
