Commit message: camera in and wheels oriented correctly

File: xacro/bobble.urdf.xacro (robot description, xacro)
@@ -2,7 +2,5 @@
 <robot name="bobblebot" xmlns:xacro="http://www.ros.org/wiki/xacro">
   <xacro:include filename="$(find bobble_description)/xacro/bobble_chassis.urdf.xacro" />
-  <!--
   <xacro:include filename="$(find bobble_description)/xacro/camera.urdf.xacro" />
-  -->
   <xacro:include filename="$(find bobble_description)/xacro/bno055_imu.urdf.xacro" />
   <xacro:include filename="$(find bobble_description)/xacro/left_wheel.urdf.xacro" />

File: xacro/left_wheel.urdf.xacro (robot description, xacro)
@@ -4,4 +4,5 @@
 	<link name="left_wheel_link">
 		<inertial>
+			<origin xyz="0.0 0.0 0.0" rpy="0.0 0.0 ${pi}"/>
 			<mass value="0.084"/>
 			<inertia ixx="0.00035" ixy="0.0" ixz="0.0" iyy="0.00035" iyz="0.0" izz="0.00035"/>

File: xacro/right_wheel.urdf.xacro (robot description, xacro)
@@ -4,4 +4,5 @@
 	<link name="right_wheel_link">
 		<inertial>
+			<origin xyz="0.0 0.0 0.0" rpy="0.0 0.0 ${pi}"/>
 			<mass value="0.084"/>
 			<inertia ixx="0.00035" ixy="0.0" ixz="0.0" iyy="0.00035" iyz="0.0" izz="0.00035"/>

Commit message: Try out realsense camera plugin

File: xacro/bobble.urdf.xacro (robot description, xacro)
@@ -2,5 +2,5 @@
 <robot name="bobblebot" xmlns:xacro="http://www.ros.org/wiki/xacro">
   <xacro:include filename="$(find bobble_description)/xacro/bobble_chassis.urdf.xacro" />
-  <xacro:include filename="$(find bobble_description)/xacro/camera.urdf.xacro" />
+  <xacro:include filename="$(find realsense_gazebo_plugin)/urdf/realsense-RS200.macro.xacro"/>
   <xacro:include filename="$(find bobble_description)/xacro/bno055_imu.urdf.xacro" />
   <xacro:include filename="$(find bobble_description)/xacro/left_wheel.urdf.xacro" />
@@ -8,6 +8,7 @@
   <xacro:bobble_chassis>
   </xacro:bobble_chassis>
-  <xacro:camera_macro parent="bobble_chassis_link">
-  </xacro:camera_macro>
+  <xacro:realsense-rs200 prefix="" parent="bobble_chassis_link">
+    <origin xyz="0 0 0.225" rpy="0 0 0" />
+  </xacro:realsense-rs200>
   <xacro:bno055_imu parent="bobble_chassis_link">
   </xacro:bno055_imu>

Commit message: added new stls for visualization

File: xacro/bobble.urdf.xacro (robot description, xacro)
@@ -2,4 +2,8 @@
 <robot name="bobblebot" xmlns:xacro="http://www.ros.org/wiki/xacro">
   <xacro:include filename="$(find bobble_description)/xacro/bobble_chassis.urdf.xacro" />
+  <xacro:include filename="$(find bobble_description)/xacro/bobble_chassis2.urdf.xacro" />
+  <xacro:include filename="$(find bobble_description)/xacro/bobble_battery.urdf.xacro" />
+  <xacro:include filename="$(find bobble_description)/xacro/bobble_realsense.urdf.xacro" />
+  <xacro:include filename="$(find bobble_description)/xacro/bobble_electronics.urdf.xacro" />
   <xacro:include filename="$(find bobble_description)/xacro/camera.urdf.xacro" />
   <xacro:include filename="$(find bobble_description)/xacro/bno055_imu.urdf.xacro" />
@@ -8,8 +12,16 @@
   <xacro:bobble_chassis>
   </xacro:bobble_chassis>
-  <xacro:camera_macro parent="bobble_chassis_link">
-  </xacro:camera_macro>
+  <xacro:bobble_chassis2 parent="bobble_chassis_link">
+  </xacro:bobble_chassis2>
+  <xacro:bobble_battery parent="bobble_chassis_link">
+  </xacro:bobble_battery>
+  <xacro:bobble_realsense parent="bobble_chassis_link">
+  </xacro:bobble_realsense>
+  <xacro:bobble_electronics parent="bobble_chassis_link">
+  </xacro:bobble_electronics>
   <xacro:bno055_imu parent="bobble_chassis_link">
   </xacro:bno055_imu>
+  <!--<xacro:camera_macro parent="bobble_chassis_link">
+  </xacro:camera_macro>-->
   <xacro:left_wheel parent="bobble_chassis_link">
   </xacro:left_wheel>

File: xacro/bobble_chassis.urdf.xacro (robot description, xacro)
@@ -1,3 +1,4 @@
 <?xml version="1.0" ?>
+<!-- This xacro file contains visual elements only -->
 <robot xmlns:xacro="http://www.ros.org/wiki/xacro">
   <xacro:macro name="bobble_chassis">
@@ -8,12 +9,12 @@
 	  		<inertia ixx="0.03" ixy="0.0" ixz="0.0" iyy="0.03" iyz="0.0" izz="0.03"/>
 		</inertial>
-		<visual>
-	  		<origin xyz="-0.05862 0.09227 -0.022" rpy="1.5707 0.0 0.0"/>
+        <visual>
+            <origin xyz="0.0 0.0 0.0" rpy="0.0 0.0 0.0"/>
             <geometry>
-  				<mesh filename="package://bobble_description/meshes/chassis.dae" scale="0.001 0.001 0.001"/>
+  				<mesh filename="package://bobble_description/meshes/chassis_grey.stl" scale="0.001 0.001 0.001"/>
             </geometry>
-   		</visual>
+        </visual>
 		<collision>
-	  		<origin xyz="0.0 0.0 0.10263" rpy="0.0 0.0 0.0"/>
+            <origin xyz="0.0 0.0 0.10263" rpy="0.0 0.0 0.0"/>
             <geometry>
               <box size="0.122 0.1129 0.19226" />
@@ -24,4 +25,7 @@
 	<gazebo reference="bobble_chassis_link">
 		<selfCollide>false</selfCollide>
+        <material>
+            Gazebo/Gray
+        </material>
 	</gazebo>
 	</xacro:macro>

File: xacro/left_wheel.urdf.xacro (robot description, xacro)
@@ -1,4 +1,5 @@
 <?xml version="1.0" ?>
 <robot xmlns:xacro="http://www.ros.org/wiki/xacro">
+    <xacro:include filename="$(find bobble_description)/xacro/materials/materials.xacro" />
   <xacro:macro name="left_wheel" params="parent">
 	<link name="left_wheel_link">
@@ -9,8 +10,9 @@
 		</inertial>
 		<visual>
-			<origin xyz="-0.0275 -0.0135 -0.0275" rpy="0.0 0.0 0.0"/>
+            <origin xyz="0.0 0.0 0.0" rpy="0.0 0.0 0.0"/>
 			<geometry name="left_wheel_link_visual">
-  				<mesh filename="package://bobble_description/meshes/wheel.dae" scale="0.001 0.001 0.001"/>
+  				<mesh filename="package://bobble_description/meshes/wheel.stl" scale="0.001 0.001 0.001"/>
 			</geometry>
+            <material name="Orange"/>
   		</visual>
 		<collision>
@@ -24,9 +26,10 @@
 	<gazebo reference="left_wheel_link">
 		<selfCollide>false</selfCollide>
+        <material>Gazebo/Orange</material>
 	</gazebo>
 	<joint name="left_wheel_hinge" type="continuous">
 		<parent link="${parent}"/>
 		<child link="left_wheel_link"/>
-		<origin rpy="0 0 0" xyz="0.0 0.06995 0.01375"/>
+		<origin rpy="0 0 0" xyz="0.0 0.05645 0.0"/>
 		<axis xyz="0 1 0"/>
 		<!-- <safety_controller k_velocity="0.5"/> -->

File: xacro/right_wheel.urdf.xacro (robot description, xacro)
@@ -1,4 +1,5 @@
 <?xml version="1.0" ?>
 <robot xmlns:xacro="http://www.ros.org/wiki/xacro">
+  <xacro:include filename="$(find bobble_description)/xacro/materials/materials.xacro" />
   <xacro:macro name="right_wheel" params="parent">
 	<link name="right_wheel_link">
@@ -9,8 +10,9 @@
 		</inertial>
 		<visual>
-			<origin xyz="0.0275 0.0135 -0.0275" rpy="0.0 0.0 3.1415926"/>
-			<geometry name="right_wheel_link_visual">
-  				<mesh filename="package://bobble_description/meshes/wheel.dae" scale="0.001 0.001 0.001"/>
+            <origin xyz="0.0 0.0 0.0" rpy="0.0 0.0 ${pi}"/>
+			<geometry name="left_wheel_link_visual">
+  				<mesh filename="package://bobble_description/meshes/wheel.stl" scale="0.001 0.001 0.001"/>
 			</geometry>
+            <material name="Orange"/>
   		</visual>
 		<collision>
@@ -24,9 +26,10 @@
 	<gazebo reference="right_wheel_link">
 		<selfCollide>false</selfCollide>
+        <material>Gazebo/Orange</material>
 	</gazebo>
 	<joint name="right_wheel_hinge" type="continuous">
 		<parent link="${parent}"/>
 		<child link="right_wheel_link"/>
-		<origin rpy="0 0 0" xyz="0.0 -0.06995 0.01375"/>
+		<origin rpy="0 0 0" xyz="0.0 -0.05645 0.0"/>
 		<axis xyz="0 1 0"/>
 		<!-- <safety_controller k_velocity="0.5"/> -->

Commit message: Update package for ROS2 migration: change CMake minimum version, update package.xml format and dependencies, convert launch files to Python, and add migration plan documentation. Also, adjust mesh file paths in URDFs for compatibility.

File: xacro/bobble.urdf.xacro (robot description, xacro)
@@ -29,18 +29,18 @@
   </xacro:right_wheel>
   <gazebo>
-    <plugin name="gazebo_ros_control" filename="libgazebo_ros_control.so" >
-      <robotNamespace>/bobble</robotNamespace>
-      <robotSimType>gazebo_ros_control/DefaultRobotHWSim</robotSimType>
-      <controlPeriod>0.002</controlPeriod>
-      <legacyModeNS>false</legacyModeNS>
+    <plugin filename="libgazebo_ros2_control.so" name="gazebo_ros2_control">
+      <parameters>$(find bobble_description)/config/ros2_controllers.yaml</parameters>
+      <ros>
+        <namespace>/bobble</namespace>
+      </ros>
     </plugin>
-    <plugin name='gazebo_ros_imu' filename='libhector_gazebo_ros_imu.so'>
-      <alwaysOn>true</alwaysOn>
-      <updateRate>200.0</updateRate>
+    <plugin name="imu_plugin" filename="libgazebo_ros_imu_sensor.so">
       <bodyName>bno055_imu_link</bodyName>
       <topicName>/imu_bosch/data_raw</topicName>
+      <updateRate>200.0</updateRate>
       <gaussianNoise>0.02</gaussianNoise>
-      <xyzOffsets>0 0 0</xyzOffsets>
-      <rpyOffsets>0 0 0</rpyOffsets>
+      <ros>
+        <namespace>/bobble</namespace>
+      </ros>
     </plugin>
   </gazebo>

File: xacro/bobble_battery.urdf.xacro (robot description, xacro)
@@ -14,5 +14,5 @@
             <origin xyz="0.0 0.0 0.0" rpy="0.0 0.0 0.0"/>
 			  <geometry>
-  				  <mesh filename="package://bobble_description/meshes/battery.stl" scale="0.001 0.001 0.001"/>
+  				  <mesh filename="$(find bobble_description)/meshes/battery.stl" scale="0.001 0.001 0.001"/>
 			  </geometry>
 			  <material name="black"/>

File: xacro/bobble_chassis.urdf.xacro (robot description, xacro)
@@ -12,5 +12,5 @@
             <origin xyz="0.0 0.0 0.0" rpy="0.0 0.0 0.0"/>
             <geometry>
-  				<mesh filename="package://bobble_description/meshes/chassis_grey.stl" scale="0.001 0.001 0.001"/>
+  				<mesh filename="$(find bobble_description)/meshes/chassis_grey.stl" scale="0.001 0.001 0.001"/>
             </geometry>
         </visual>

File: xacro/bobble_chassis2.urdf.xacro (robot description, xacro)
@@ -14,5 +14,5 @@
             <origin xyz="0.0 0.0 0.0" rpy="0.0 0.0 0.0"/>
 			  <geometry>
-  				  <mesh filename="package://bobble_description/meshes/chassis_orange.stl" scale="0.001 0.001 0.001"/>
+  				  <mesh filename="$(find bobble_description)/meshes/chassis_orange.stl" scale="0.001 0.001 0.001"/>
 			  </geometry>
 			  <material name="orange"/>

File: xacro/bobble_electronics.urdf.xacro (robot description, xacro)
@@ -13,5 +13,5 @@
             <origin xyz="0.0 0.0 0.0" rpy="0.0 0.0 0.0"/>
 			  <geometry>
-                      <mesh filename="package://bobble_description/meshes/electronics.stl" scale="0.001 0.001 0.001"/>
+                      <mesh filename="$(find bobble_description)/meshes/electronics.stl" scale="0.001 0.001 0.001"/>
 			  </geometry>
 			  <material name="green"/>

File: xacro/bobble_realsense.urdf.xacro (robot description, xacro)
@@ -13,5 +13,5 @@
             <origin xyz="0.0 0.0 0.0" rpy="0.0 0.0 0.0"/>
 			  <geometry>
-  				  <mesh filename="package://bobble_description/meshes/realsense.stl" scale="0.001 0.001 0.001"/>
+  				  <mesh filename="$(find bobble_description)/meshes/realsense.stl" scale="0.001 0.001 0.001"/>
 			  </geometry>
 			  <material name="gray"/>

File: xacro/camera.urdf.xacro (robot description, xacro)
@@ -50,16 +50,12 @@
 			  </camera>
 			  <plugin name="camera_controller" filename="libgazebo_ros_camera.so">
-				  <alwaysOn>true</alwaysOn>
-				  <updateRate>0.0</updateRate>
-				  <cameraName>bobble_bot/camera</cameraName>
-				  <imageTopicName>image_raw</imageTopicName>
-				  <cameraInfoTopicName>camera_info</cameraInfoTopicName>
-				  <frameName>camera_link</frameName>
-				  <hackBaseline>0.07</hackBaseline>
-				  <distortionK1>0.0</distortionK1>
-				  <distortionK2>0.0</distortionK2>
-				  <distortionK3>0.0</distortionK3>
-				  <distortionT1>0.0</distortionT1>
-				  <distortionT2>0.0</distortionT2>
+				  <ros>
+					  <namespace>/bobble</namespace>
+					  <remapping>~/image_raw:=camera/image_raw</remapping>
+					  <remapping>~/camera_info:=camera/camera_info</remapping>
+				  </ros>
+				  <camera_name>camera</camera_name>
+				  <frame_name>camera_link</frame_name>
+				  <hack_baseline>0.07</hack_baseline>
 			  </plugin>
 		  </sensor>

File: xacro/left_wheel.urdf.xacro (robot description, xacro)
@@ -12,5 +12,5 @@
             <origin xyz="0.0 0.0 0.0" rpy="0.0 0.0 0.0"/>
 			<geometry name="left_wheel_link_visual">
-  				<mesh filename="package://bobble_description/meshes/wheel.stl" scale="0.001 0.001 0.001"/>
+  				<mesh filename="$(find bobble_description)/meshes/wheel.stl" scale="0.001 0.001 0.001"/>
 			</geometry>
             <material name="Orange"/>

File: xacro/right_wheel.urdf.xacro (robot description, xacro)
@@ -12,5 +12,5 @@
             <origin xyz="0.0 0.0 0.0" rpy="0.0 0.0 ${pi}"/>
 			<geometry name="left_wheel_link_visual">
-  				<mesh filename="package://bobble_description/meshes/wheel.stl" scale="0.001 0.001 0.001"/>
+  				<mesh filename="$(find bobble_description)/meshes/wheel.stl" scale="0.001 0.001 0.001"/>
 			</geometry>
             <material name="Orange"/>
