Commit message: Add installation of params directory and update README with detailed package information and usage examples. Refactor launch files for improved world file validation and error handling. Update URDF mesh paths for compatibility.

File: xacro/bno055_imu.urdf.xacro (robot description, xacro)
@@ -21,7 +21,4 @@
 		</collision>
 	</link>
-	<gazebo reference="bno055_imu_link">
-		<selfCollide>false</selfCollide>
-	</gazebo>
 	<joint name="bno055_imu_joint" type="fixed">
 		<parent link="${parent}"/>

File: xacro/bobble.urdf.xacro (robot description, xacro)
@@ -10,4 +10,5 @@
   <xacro:include filename="$(find bobble_description)/xacro/left_wheel.urdf.xacro" />
   <xacro:include filename="$(find bobble_description)/xacro/right_wheel.urdf.xacro" />
+  <xacro:include filename="$(find bobble_description)/xacro/bobble.gazebo" />
   <xacro:bobble_chassis>
   </xacro:bobble_chassis>
@@ -28,20 +29,3 @@
   <xacro:right_wheel parent="bobble_chassis_link">
   </xacro:right_wheel>
-  <gazebo>
-    <plugin filename="libgazebo_ros2_control.so" name="gazebo_ros2_control">
-      <parameters>$(find bobble_description)/config/ros2_controllers.yaml</parameters>
-      <ros>
-        <namespace>/bobble</namespace>
-      </ros>
-    </plugin>
-    <plugin name="imu_plugin" filename="libgazebo_ros_imu_sensor.so">
-      <bodyName>bno055_imu_link</bodyName>
-      <topicName>/imu_bosch/data_raw</topicName>
-      <updateRate>200.0</updateRate>
-      <gaussianNoise>0.02</gaussianNoise>
-      <ros>
-        <namespace>/bobble</namespace>
-      </ros>
-    </plugin>
-  </gazebo>
 </robot>

File: xacro/bobble_battery.urdf.xacro (robot description, xacro)
@@ -14,5 +14,5 @@
             <origin xyz="0.0 0.0 0.0" rpy="0.0 0.0 0.0"/>
 			  <geometry>
-  				  <mesh filename="$(find bobble_description)/meshes/battery.stl" scale="0.001 0.001 0.001"/>
+  				  <mesh filename="file://$(find bobble_description)/meshes/battery.stl" scale="0.001 0.001 0.001"/>
 			  </geometry>
 			  <material name="black"/>

File: xacro/bobble_chassis.urdf.xacro (robot description, xacro)
@@ -12,5 +12,5 @@
             <origin xyz="0.0 0.0 0.0" rpy="0.0 0.0 0.0"/>
             <geometry>
-  				<mesh filename="$(find bobble_description)/meshes/chassis_grey.stl" scale="0.001 0.001 0.001"/>
+  				<mesh filename="file://$(find bobble_description)/meshes/chassis_grey.stl" scale="0.001 0.001 0.001"/>
             </geometry>
         </visual>

File: xacro/bobble_chassis2.urdf.xacro (robot description, xacro)
@@ -14,5 +14,5 @@
             <origin xyz="0.0 0.0 0.0" rpy="0.0 0.0 0.0"/>
 			  <geometry>
-  				  <mesh filename="$(find bobble_description)/meshes/chassis_orange.stl" scale="0.001 0.001 0.001"/>
+  				  <mesh filename="file://$(find bobble_description)/meshes/chassis_orange.stl" scale="0.001 0.001 0.001"/>
 			  </geometry>
 			  <material name="orange"/>

File: xacro/bobble_electronics.urdf.xacro (robot description, xacro)
@@ -13,5 +13,5 @@
             <origin xyz="0.0 0.0 0.0" rpy="0.0 0.0 0.0"/>
 			  <geometry>
-                      <mesh filename="$(find bobble_description)/meshes/electronics.stl" scale="0.001 0.001 0.001"/>
+                      <mesh filename="file://$(find bobble_description)/meshes/electronics.stl" scale="0.001 0.001 0.001"/>
 			  </geometry>
 			  <material name="green"/>

File: xacro/bobble_realsense.urdf.xacro (robot description, xacro)
@@ -13,5 +13,5 @@
             <origin xyz="0.0 0.0 0.0" rpy="0.0 0.0 0.0"/>
 			  <geometry>
-  				  <mesh filename="$(find bobble_description)/meshes/realsense.stl" scale="0.001 0.001 0.001"/>
+  				  <mesh filename="file://$(find bobble_description)/meshes/realsense.stl" scale="0.001 0.001 0.001"/>
 			  </geometry>
 			  <material name="gray"/>

File: xacro/left_wheel.urdf.xacro (robot description, xacro)
@@ -12,5 +12,5 @@
             <origin xyz="0.0 0.0 0.0" rpy="0.0 0.0 0.0"/>
 			<geometry name="left_wheel_link_visual">
-  				<mesh filename="$(find bobble_description)/meshes/wheel.stl" scale="0.001 0.001 0.001"/>
+  				<mesh filename="file://$(find bobble_description)/meshes/wheel.stl" scale="0.001 0.001 0.001"/>
 			</geometry>
             <material name="Orange"/>

File: xacro/right_wheel.urdf.xacro (robot description, xacro)
@@ -12,5 +12,5 @@
             <origin xyz="0.0 0.0 0.0" rpy="0.0 0.0 ${pi}"/>
 			<geometry name="left_wheel_link_visual">
-  				<mesh filename="$(find bobble_description)/meshes/wheel.stl" scale="0.001 0.001 0.001"/>
+  				<mesh filename="file://$(find bobble_description)/meshes/wheel.stl" scale="0.001 0.001 0.001"/>
 			</geometry>
             <material name="Orange"/>
