Commit message: updated the hinge location for correct behavior
Former-commit-id: 1c88df36b83fe977c4b5878017cfa39d8e527ea7

File: xacro/left_wheel.urdf.xacro (robot description, xacro)
@@ -8,5 +8,5 @@
 		</inertial>
 		<visual>
-			<origin xyz="0.0 0.1 0.05" rpy="0.0 1.5707 1.5707"/>
+			<origin xyz="0.0 0.0 0.0" rpy="0.0 1.5707 1.5707"/>
 			<geometry name="left_wheel_link_visual">
   				<mesh filename="package://bobble_description/meshes/wheel.dae" scale="1.0 1.0 1.0"/>
@@ -14,5 +14,5 @@
   		</visual>
 		<collision>
-			<origin xyz="0.0 0.1 0.05" rpy="0.0 1.5707 1.5707"/>
+			<origin xyz="0.0 0.0 0.0" rpy="0.0 1.5707 1.5707"/>
             <geometry>
               <cylinder radius="0.05" length="0.05" />
@@ -27,7 +27,7 @@
 		<parent link="${parent}"/>
 		<child link="left_wheel_link"/>
-		<origin rpy="0 0 0" xyz="0.0 0.0 0.0"/>
+		<origin rpy="0 0 0" xyz="0.0 0.1 0.05"/>
 		<axis xyz="0 1 0"/>
-		<limit effort="30" lower="-2.6" upper="2.6" velocity="2.0"/>
+		<limit effort="30" lower="-1000.0" upper="1000.0" velocity="2.0"/>
 		<!-- <safety_controller k_velocity="0.5"/> -->
 		<!-- <joint_properties damping="100.0" friction="1000.0" /> -->

File: xacro/right_wheel.urdf.xacro (robot description, xacro)
@@ -8,5 +8,5 @@
 		</inertial>
 		<visual>
-			<origin xyz="0.0 -0.1 0.05" rpy="0.0 1.5707 -1.5707"/>
+			<origin xyz="0.0 0.0 0.0" rpy="0.0 1.5707 -1.5707"/>
 			<geometry name="right_wheel_link_visual">
   				<mesh filename="package://bobble_description/meshes/wheel.dae" scale="1.0 1.0 1.0"/>
@@ -14,5 +14,5 @@
   		</visual>
 		<collision>
-			<origin xyz="0.0 -0.1 0.05" rpy="0.0 1.5707 -1.5707"/>
+			<origin xyz="0.0 0.0 0.0" rpy="0.0 1.5707 -1.5707"/>
             <geometry>
               <cylinder radius="0.05" length="0.05" />
@@ -27,7 +27,7 @@
 		<parent link="${parent}"/>
 		<child link="right_wheel_link"/>
-		<origin rpy="0 0 0" xyz="0.0 0.0 0.0"/>
+		<origin rpy="0 0 0" xyz="0.0 -0.1 0.05"/>
 		<axis xyz="0 1 0"/>
-		<limit effort="30" lower="-2.6" upper="2.6" velocity="2.0"/>
+		<limit effort="30" lower="-1000.0" upper="1000.0" velocity="2.0"/>
 		<!-- <safety_controller k_velocity="0.5"/> -->
 		<!-- <joint_properties damping="100.0" friction="1000.0" /> -->

Commit message: Update README to reflect new maintainer and enhance clarity on package contributions. Modify left and right wheel URDF files to improve contact coefficients and dynamics parameters for better simulation performance.

File: xacro/left_wheel.urdf.xacro (robot description, xacro)
@@ -21,5 +21,5 @@
               <cylinder radius="0.0275" length="0.027" />
             </geometry>
-			<contact_coefficients kd="1.0" kp="1000.0" mu="0"/>
+			<contact_coefficients kd="1.0" kp="1000.0" mu="1.0"/>
 		</collision>
 	</link>
@@ -27,4 +27,10 @@
 		<selfCollide>false</selfCollide>
         <material>Gazebo/Orange</material>
+        <mu1>1.0</mu1>
+        <mu2>1.0</mu2>
+        <kp>500000.0</kp>
+        <kd>10.0</kd>
+        <minDepth>0.001</minDepth>
+        <maxVel>0.1</maxVel>
 	</gazebo>
 	<joint name="left_wheel_hinge" type="continuous">
@@ -35,5 +41,5 @@
 		<!-- <safety_controller k_velocity="0.5"/> -->
 		<!-- <joint_properties damping="100.0" friction="1000.0" /> -->
-    	<dynamics damping="0.0" friction="0.0"/>
+    	<dynamics damping="0.1" friction="0.1"/>
 	</joint>
 	<transmission name="left_wheel_transmission">

File: xacro/right_wheel.urdf.xacro (robot description, xacro)
@@ -21,5 +21,5 @@
               <cylinder radius="0.0275" length="0.027" />
             </geometry>
-			<contact_coefficients kd="1.0" kp="1000.0" mu="0"/>
+			<contact_coefficients kd="1.0" kp="1000.0" mu="1.0"/>
 		</collision>
 	</link>
@@ -27,4 +27,10 @@
 		<selfCollide>false</selfCollide>
         <material>Gazebo/Orange</material>
+        <mu1>1.0</mu1>
+        <mu2>1.0</mu2>
+        <kp>500000.0</kp>
+        <kd>10.0</kd>
+        <minDepth>0.001</minDepth>
+        <maxVel>0.1</maxVel>
 	</gazebo>
 	<joint name="right_wheel_hinge" type="continuous">
@@ -35,5 +41,5 @@
 		<!-- <safety_controller k_velocity="0.5"/> -->
 		<!-- <joint_properties damping="100.0" friction="1000.0" /> -->
-		<dynamics damping="0.0" friction="0.0"/>
+		<dynamics damping="0.1" friction="0.1"/>
 	</joint>
 	<transmission name="right_wheel_transmission">
